File: ssr.sch (KiCad schematic (older format))
At the start: 29 parts, among them CON1 AVR-ISP-6, IC1 ATTINY44-SS, P1 CONN_4, P2 CONTACT, P3 CONTACT, P4 CONTACT, P6 CONN_4, Q1 MOSFET_N, U1 MOC-3052, U2 TRIAC, U3 LTV-814

Commit message: boards sent for manufacture
Parts:
- added C6: C, ~, symbol C
- added D1, D2: LED, ~, symbol LED
- added R11, R12: R, symbol R
Connections:
- wire segments 69 -> 78
Changed lines of the file:
@@
-EESchema Schematic File Version 2  date Fri 26 Apr 2013 07:25:16 PM CEST
+EESchema Schematic File Version 2  date Tue 07 May 2013 10:19:57 PM CEST
 LIBS:power
 LIBS:device
@@
 Sheet 1 1
 Title ""
-Date "24 apr 2013"
+Date "3 may 2013"
 Rev ""
 Comp ""
@@
 $EndComp
 $Comp
-L VCC #PWR12
+L VCC #PWR01
 U 1 1 511F836F
 P 4850 3450
-F 0 "#PWR12" H 4850 3550 30  0001 C CNN
+F 0 "#PWR01" H 4850 3550 30  0001 C CNN
 F 1 "VCC" H 4850 3550 30  0000 C CNN
 F 2 "" H 4850 3450 60  0000 C CNN
@@
 $EndComp
 $Comp
-L VCC #PWR9
+L VCC #PWR02
 U 1 1 511F856B
 P 4450 3400
-F 0 "#PWR9" H 4450 3500 30  0001 C CNN
+F 0 "#PWR02" H 4450 3500 30  0001 C CNN
 F 1 "VCC" H 4450 3500 30  0000 C CNN
 F 2 "" H 4450 3400 60  0000 C CNN
@@
 $EndComp
 $Comp
-L GND #PWR8
+L GND #PWR03
 U 1 1 511F857A
 P 3900 3200
-F 0 "#PWR8" H 3900 3200 30  0001 C CNN
+F 0 "#PWR03" H 3900 3200 30  0001 C CNN
 F 1 "GND" H 3900 3130 30  0001 C CNN
 F 2 "" H 3900 3200 60  0000 C CNN
@@
 ZERO_CROSSING
 $Comp
-L GND #PWR4
+L GND #PWR04
 U 1 1 511F87D7
 P 2300 3150
-F 0 "#PWR4" H 2300 3150 30  0001 C CNN
+F 0 "#PWR04" H 2300 3150 30  0001 C CNN
 F 1 "GND" H 2300 3080 30  0001 C CNN
 F 2 "" H 2300 3150 60  0000 C CNN
@@
 $EndComp
 $Comp
-L GND #PWR15
+L GND #PWR05
 U 1 1 5165DEAF
 P 4950 4600
-F 0 "#PWR15" H 4950 4600 30  0001 C CNN
+F 0 "#PWR05" H 4950 4600 30  0001 C CNN
 F 1 "GND" H 4950 4530 30  0001 C CNN
 F 2 "" H 4950 4600 60  0000 C CNN
@@
 $EndComp
 $Comp
-L VCC #PWR1
+L VCC #PWR06
 U 1 1 51697FD8
 P 550 3900
-F 0 "#PWR1" H 550 4000 30  0001 C CNN
+F 0 "#PWR06" H 550 4000 30  0001 C CNN
 F 1 "VCC" H 550 4000 30  0000 C CNN
 F 2 "" H 550 3900 60  0000 C CNN
@@
 $EndComp
 $Comp
-L GND #PWR2
+L GND #PWR07
 U 1 1 51697FDE
 P 550 5200
-F 0 "#PWR2" H 550 5200 30  0001 C CNN
+F 0 "#PWR07" H 550 5200 30  0001 C CNN
 F 1 "GND" H 550 5130 30  0001 C CNN
 F 2 "" H 550 5200 60  0000 C CNN
@@
 $EndComp
 $Comp
-L VCC #PWR10
+L VCC #PWR08
 U 1 1 51698026
-P 4650 4800
-F 0 "#PWR10" H 4650 4900 30  0001 C CNN
-F 1 "VCC" H 4650 4900 30  0000 C CNN
-F 2 "" H 4650 4800 60  0000 C CNN
-F 3 "" H 4650 4800 60  0000 C CNN
-	1    4650 4800
-	1    0    0    -1
-$EndComp
-$Comp
-L GND #PWR11
+P 4500 5200
+F 0 "#PWR08" H 4500 5300 30  0001 C CNN
+F 1 "VCC" H 4500 5300 30  0000 C CNN
+F 2 "" H 4500 5200 60  0000 C CNN
+F 3 "" H 4500 5200 60  0000 C CNN
+	1    4500 5200
+	1    0    0    -1
+$EndComp
+$Comp
+L GND #PWR09
 U 1 1 5169802C
-P 4650 5200
-F 0 "#PWR11" H 4650 5200 30  0001 C CNN
-F 1 "GND" H 4650 5130 30  0001 C CNN
-F 2 "" H 4650 5200 60  0000 C CNN
-F 3 "" H 4650 5200 60  0000 C CNN
-	1    4650 5200
+P 4500 4750
+F 0 "#PWR09" H 4500 4750 30  0001 C CNN
+F 1 "GND" H 4500 4680 30  0001 C CNN
+F 2 "" H 4500 4750 60  0000 C CNN
+F 3 "" H 4500 4750 60  0000 C CNN
+	1    4500 4750
 	1    0    0    -1
 $EndComp
@@
 $EndComp
 $Comp
-L VCC #PWR5
+L VCC #PWR010
 U 1 1 516986F1
 P 2800 5600
-F 0 "#PWR5" H 2800 5700 30  0001 C CNN
+F 0 "#PWR010" H 2800 5700 30  0001 C CNN
 F 1 "VCC" H 2800 5700 30  0000 C CNN
 F 2 "" H 2800 5600 60  0000 C CNN
@@
 $EndComp
 $Comp
-L VCC #PWR6
+L VCC #PWR011
 U 1 1 516A4D45
 P 3775 5975
-F 0 "#PWR6" H 3775 6075 30  0001 C CNN
+F 0 "#PWR011" H 3775 6075 30  0001 C CNN
 F 1 "VCC" H 3775 6075 30  0000 C CNN
 F 2 "" H 3775 5975 60  0000 C CNN
@@
 $EndComp
 $Comp
-L GND #PWR7
+L GND #PWR012
 U 1 1 516A4D4B
 P 3775 6450
-F 0 "#PWR7" H 3775 6450 30  0001 C CNN
+F 0 "#PWR012" H 3775 6450 30  0001 C CNN
 F 1 "GND" H 3775 6380 30  0001 C CNN
 F 2 "" H 3775 6450 60  0000 C CNN
@@
 $EndComp
 $Comp
-L VCC #PWR13
+L VCC #PWR013
 U 1 1 516A5040
 P 4850 5650
-F 0 "#PWR13" H 4850 5750 30  0001 C CNN
+F 0 "#PWR013" H 4850 5750 30  0001 C CNN
 F 1 "VCC" H 4850 5750 30  0000 C CNN
 F 2 "" H 4850 5650 60  0000 C CNN
@@
 $EndComp
 $Comp
-L GND #PWR14
+L GND #PWR014
 U 1 1 516A5046
 P 4850 6050
-F 0 "#PWR14" H 4850 6050 30  0001 C CNN
+F 0 "#PWR014" H 4850 6050 30  0001 C CNN
 F 1 "GND" H 4850 5980 30  0001 C CNN
 F 2 "" H 4850 6050 60  0000 C CNN
@@
 $EndComp
 $Comp
-L VCC #PWR3
+L VCC #PWR015
 U 1 1 516B0796
 P 2300 1300
-F 0 "#PWR3" H 2300 1400 30  0001 C CNN
+F 0 "#PWR015" H 2300 1400 30  0001 C CNN
 F 1 "VCC" H 2300 1400 30  0000 C CNN
 F 2 "" H 2300 1300 60  0000 C CNN
@@
 Connection ~ 3250 3300
 Wire Wire Line
-	2650 4100 3250 4100
-Wire Wire Line
-	2650 4200 3300 4200
-Wire Wire Line
-	3300 4200 3300 3500
+	3300 3500 3300 5000
 Wire Wire Line
 	3200 3500 3550 3500
@@
 	1800 2400 2000 2400
 Wire Wire Line
-	3250 4100 3250 3300
+	3250 3300 3250 4600
+$Comp
+L C C6
+U 1 1 5183F45A
+P 2000 1600
+F 0 "C6" H 2000 1700 40  0000 L CNN
+F 1 "C" H 2006 1515 40  0000 L CNN
+F 2 "~" H 2038 1450 30  0000 C CNN
+F 3 "~" H 2000 1600 60  0000 C CNN
+	1    2000 1600
+	1    0    0    -1
+$EndComp
+Wire Wire Line
+	2300 1400 2000 1400
+$Comp
+L GND #PWR016
+U 1 1 5183F4C0
+P 2000 1800
+F 0 "#PWR016" H 2000 1800 30  0001 C CNN
+F 1 "GND" H 2000 1730 30  0001 C CNN
+F 2 "" H 2000 1800 60  0000 C CNN
+F 3 "" H 2000 1800 60  0000 C CNN
+	1    2000 1800
+	1    0    0    -1
+$EndComp
+Wire Wire Line
+	4500 5200 4650 5200
+Wire Wire Line
+	4500 4750 4500 4650
+Wire Wire Line
+	4500 4650 4650 4650
+Wire Wire Line
+	4650 4650 4650 4800
+Wire Wire Line
+	3300 5000 2650 5000
+Wire Wire Line
+	3250 4600 2650 4600
+$Comp
+L LED D1
+U 1 1 51840F81
+P 3150 5350
+F 0 "D1" H 3150 5450 50  0000 C CNN
+F 1 "LED" H 3150 5250 50  0000 C CNN
+F 2 "~" H 3150 5350 60  0000 C CNN
+F 3 "~" H 3150 5350 60  0000 C CNN
+	1    3150 5350
+	0    1    1    0
+$EndComp
+$Comp
+L GND #PWR017
+U 1 1 51840F90
+P 3150 5550
+F 0 "#PWR017" H 3150 5550 30  0001 C CNN
+F 1 "GND" H 3150 5480 30  0001 C CNN
+F 2 "" H 3150 5550 60  0000 C CNN
+F 3 "" H 3150 5550 60  0000 C CNN
+	1    3150 5550
+	1    0    0    -1
+$EndComp
+$Comp
+L LED D2
+U 1 1 51840FAE
+P 3300 5350
+F 0 "D2" H 3300 5450 50  0000 C CNN
+F 1 "LED" H 3300 5250 50  0000 C CNN
+F 2 "~" H 3300 5350 60  0000 C CNN
+F 3 "~" H 3300 5350 60  0000 C CNN
+	1    3300 5350
+	0    1    1    0
+$EndComp
+$Comp
+L GND #PWR018
+U 1 1 51840FB4
+P 3300 5550
+F 0 "#PWR018" H 3300 5550 30  0001 C CNN
+F 1 "GND" H 3300 5480 30  0001 C CNN
+F 2 "" H 3300 5550 60  0000 C CNN
+F 3 "" H 3300 5550 60  0000 C CNN
+	1    3300 5550
+	1    0    0    -1
+$EndComp
+$Comp
+L R R11
+U 1 1 51840FC2
+P 2900 4800
+F 0 "R11" V 2980 4800 50  0000 C CNN
+F 1 "R" V 2900 4800 50  0000 C CNN
+F 2 "" H 2900 4800 60  0000 C CNN
+F 3 "" H 2900 4800 60  0000 C CNN
+	1    2900 4800
+	0    -1   -1   0
+$EndComp
+$Comp
+L R R12
+U 1 1 51840FC9
+P 2900 4900
+F 0 "R12" V 2980 4900 50  0000 C CNN
+F 1 "R" V 2900 4900 50  0000 C CNN
+F 2 "" H 2900 4900 60  0000 C CNN
+F 3 "" H 2900 4900 60  0000 C CNN
+	1    2900 4900
+	0    -1   -1   0
+$EndComp
+Wire Wire Line
+	3150 4900 3150 5150
+Wire Wire Line
+	3150 4800 3200 4800
+Wire Wire Line
+	3200 4800 3200 5150
+Wire Wire Line
+	3200 5150 3300 5150
 $EndSCHEMATC

Commit message: some work on firmware, experiments, some documentation has been added
Parts:
- R10: value R -> 200
- R2: value 200R -> 47k
- R4, R5: value 8.2k 5W -> 16.4k
- U2: value TRIAC -> BTA41
Connections:
- net labels added: SCL, SDA
- wire segments 78 -> 97
Other:
- note added: "R = 340V / 1A\n--------------------\n(1A - opto triac max surge current)"
- note added: "TODO: move ON signal to another pin, ICP is cool for capturing timer"
- note removed: "P = 340V * 1A\n R = 340V / 1A\n--------------------\n(opto triac max surge current)"
- moved on the sheet: R2
Changed lines of the file:
@@
-EESchema Schematic File Version 2  date Tue 07 May 2013 10:19:57 PM CEST
+EESchema Schematic File Version 2
 LIBS:power
 LIBS:device
@@
 Sheet 1 1
 Title ""
-Date "3 may 2013"
+Date "13 may 2013"
 Rev ""
 Comp ""
@@
 P 5000 2000
 F 0 "U2" H 4750 2350 70  0000 C CNN
-F 1 "TRIAC" H 4700 1750 60  0000 C CNN
+F 1 "BTA41" H 4700 1750 60  0000 C CNN
 F 2 "" H 5000 2000 60  0000 C CNN
 F 3 "" H 5000 2000 60  0000 C CNN
@@
 Text Notes 7700 1500 0    60   ~ 0
 240VAC
-Text Notes 7700 2400 0    60   ~ 0
+Text Notes 7300 2400 0    60   ~ 0
 LOAD
 $Comp
@@
 P 6950 4050
 F 0 "R4" V 7030 4050 50  0000 C CNN
-F 1 "8.2k 5W" V 6950 4050 50  0000 C CNN
+F 1 "16.4k" V 6950 4050 50  0000 C CNN
 F 2 "" H 6950 4050 60  0000 C CNN
 F 3 "" H 6950 4050 60  0000 C CNN
@@
 P 6950 4350
 F 0 "R5" V 7030 4350 50  0000 C CNN
-F 1 "8.2k 5W" V 6950 4350 50  0000 C CNN
+F 1 "16.4k" V 6950 4350 50  0000 C CNN
 F 2 "" H 6950 4350 60  0000 C CNN
 F 3 "" H 6950 4350 60  0000 C CNN
@@
 L VCC #PWR01
 U 1 1 511F836F
-P 4850 3450
-F 0 "#PWR01" H 4850 3550 30  0001 C CNN
-F 1 "VCC" H 4850 3550 30  0000 C CNN
-F 2 "" H 4850 3450 60  0000 C CNN
-F 3 "" H 4850 3450 60  0000 C CNN
-	1    4850 3450
+P 5150 3450
+F 0 "#PWR01" H 5150 3550 30  0001 C CNN
+F 1 "VCC" H 5150 3550 30  0000 C CNN
+F 2 "" H 5150 3450 60  0000 C CNN
+F 3 "" H 5150 3450 60  0000 C CNN
+	1    5150 3450
 	-1   0    0    -1
 $EndComp
@@
 L R R2
 U 1 1 511F837C
-P 4850 3700
-F 0 "R2" V 4930 3700 50  0000 C CNN
-F 1 "200R" V 4850 3700 50  0000 C CNN
-F 2 "" H 4850 3700 60  0000 C CNN
-F 3 "" H 4850 3700 60  0000 C CNN
-	1    4850 3700
+P 5150 3700
+F 0 "R2" V 5230 3700 50  0000 C CNN
+F 1 "47k" V 5150 3700 50  0000 C CNN
+F 2 "" H 5150 3700 60  0000 C CNN
+F 3 "" H 5150 3700 60  0000 C CNN
+	1    5150 3700
 	1    0    0    1
 $EndComp
-Text GLabel 4750 4100 0    60   Input ~ 0
+Text GLabel 5050 4100 0    60   Input ~ 0
 ZERO_CROSSING
 $Comp
@@
 Text GLabel 1800 2400 0    60   Input ~ 0
 ON
-Text Notes 2600 950  0    60   ~ 0
-        P =  340V * 1A\n        R =  340V / 1A\n--------------------\n(opto triac max surge current)
 $Comp
 L C C3
@@
 L OPTO-TRANSISTOR-AC U3
 U 1 1 51603500
-P 5500 4250
-F 0 "U3" H 5700 4550 60  0000 C CNN
-F 1 "LTV-814" H 5600 3950 60  0000 C CNN
-F 2 "~" H 5500 4250 60  0000 C CNN
-F 3 "~" H 5500 4250 60  0000 C CNN
-	1    5500 4250
+P 5750 4250
+F 0 "U3" H 5950 4550 60  0000 C CNN
+F 1 "LTV-814" H 5850 3950 60  0000 C CNN
+F 2 "~" H 5750 4250 60  0000 C CNN
+F 3 "~" H 5750 4250 60  0000 C CNN
+	1    5750 4250
 	-1   0    0    -1
 $EndComp
@@
 L GND #PWR05
 U 1 1 5165DEAF
-P 4950 4600
-F 0 "#PWR05" H 4950 4600 30  0001 C CNN
-F 1 "GND" H 4950 4530 30  0001 C CNN
-F 2 "" H 4950 4600 60  0000 C CNN
-F 3 "" H 4950 4600 60  0000 C CNN
-	1    4950 4600
+P 5200 4550
+F 0 "#PWR05" H 5200 4550 30  0001 C CNN
+F 1 "GND" H 5200 4480 30  0001 C CNN
+F 2 "" H 5200 4550 60  0000 C CNN
+F 3 "" H 5200 4550 60  0000 C CNN
+	1    5200 4550
 	1    0    0    -1
 $EndComp
@@
 U 1 1 516976FE
 P 7200 1400
-F 0 "P2" H 7200 1300 60  0000 C CNN
-F 1 "CONTACT" H 7200 1500 60  0000 C CNN
+F 0 "P2" H 6700 1250 60  0000 C CNN
+F 1 "CONTACT" H 7000 1250 60  0000 C CNN
 F 2 "~" H 7200 1400 60  0000 C CNN
 F 3 "~" H 7200 1400 60  0000 C CNN
@@
 U 1 1 5169770B
 P 7200 1600
-F 0 "P3" H 7200 1500 60  0000 C CNN
-F 1 "CONTACT" H 7200 1700 60  0000 C CNN
+F 0 "P3" H 6700 1700 60  0000 C CNN
+F 1 "CONTACT" H 7000 1700 60  0000 C CNN
 F 2 "~" H 7200 1600 60  0000 C CNN
 F 3 "~" H 7200 1600 60  0000 C CNN
@@
 	3450 4400 3450 3200
 Wire Wire Line
-	4950 4400 3450 4400
-Wire Wire Line
-	2300 2600 2300 3150
+	5200 4400 3450 4400
+Wire Wire Line
+	2300 2600 2300 3100
+Wire Wire Line
+	2300 3100 2300 3150
 Wire Wire Line
 	3200 3400 4450 3400
 Wire Wire Line
-	6700 4350 6400 4350
-Wire Wire Line
-	6700 4050 6400 4050
+	6700 4350 6650 4350
+Wire Wire Line
+	6700 4050 6650 4050
 Wire Wire Line
 	6900 1400 6900 1750
@@
 	3550 1400 3550 1400
 Wire Wire Line
-	4850 3950 4850 4100
+	5150 3950 5150 4100
 Wire Wire Line
 	7200 3300 7200 4050
@@
 	7850 1900 7850 4350
 Wire Wire Line
-	3200 3300 3550 3300
-Wire Wire Line
-	3200 3200 3900 3200
-Connection ~ 4850 4100
-Wire Wire Line
-	4750 4100 4950 4100
+	3200 3300 3250 3300
+Wire Wire Line
+	3250 3300 3550 3300
+Wire Wire Line
+	3200 3200 3450 3200
+Wire Wire Line
+	3450 3200 3900 3200
+Connection ~ 5150 4100
+Wire Wire Line
+	5050 4100 5150 4100
+Wire Wire Line
+	5150 4100 5200 4100
 Connection ~ 7200 1900
 Connection ~ 6000 1400
@@
 	5400 2500 5400 2300
 Wire Wire Line
-	4050 2500 5500 2500
+	4050 2500 5000 2500
+Wire Wire Line
+	5000 2500 5400 2500
+Wire Wire Line
+	5400 2500 5500 2500
 Wire Wire Line
 	5000 2250 5000 2500
 Wire Wire Line
-	6100 2500 7200 2500
+	6100 2500 6700 2500
+Wire Wire Line
+	6700 2500 6900 2500
+Wire Wire Line
+	6900 2500 7200 2500
 Wire Wire Line
 	3550 1800 3550 2200
@@
 	3550 2200 4500 2200
 Wire Wire Line
-	4550 1400 6150 1400
-Wire Wire Line
-	4950 4400 4950 4600
-Wire Wire Line
-	7050 1900 7850 1900
-Wire Wire Line
-	6650 1400 7200 1400
+	4550 1400 5000 1400
+Wire Wire Line
+	5000 1400 5400 1400
+Wire Wire Line
+	5400 1400 6000 1400
+Wire Wire Line
+	6000 1400 6150 1400
+Wire Wire Line
+	5200 4400 5200 4550
+Wire Wire Line
+	7050 1900 7200 1900
+Wire Wire Line
+	7200 1900 7850 1900
+Wire Wire Line
+	6650 1400 6700 1400
+Wire Wire Line
+	6700 1400 6900 1400
+Wire Wire Line
+	6900 1400 7050 1400
+Wire Wire Line
+	7050 1400 7200 1400
 Connection ~ 7050 1400
 Wire Wire Line
@@
 Connection ~ 3450 3200
 Wire Wire Line
-	550  4750 550  5200
+	550  4750 550  5100
+Wire Wire Line
+	550  5100 550  5200
 Wire Wire Line
 	4650 5200 4650 5100
 Wire Wire Line
-	2650 4300 3400 4300
+	2650 4300 2900 4300
+Wire Wire Line
+	2900 4300 3400 4300
 Wire Wire Line
 	3400 4300 3400 4900
@@
 	3400 4900 4650 4900
 Wire Wire Line
-	2650 4400 3350 4400
-Wire Wire Line
-	3350 4400 3350 5000
+	3350 4500 3350 5000
 Wire Wire Line
 	3350 5000 4650 5000
@@
 	3300 3500 3300 5000
 Wire Wire Line
-	3200 3500 3550 3500
+	3200 3500 3300 3500
+Wire Wire Line
+	3300 3500 3550 3500
 Connection ~ 3300 3500
 Wire Wire Line
@@
 Wire Wire Line
 	2950 6100 2950 4400
-Connection ~ 2950 4400
 Wire Wire Line
 	3650 6200 3525 6200
@@
 	3000 5975 3000 4500
 Wire Wire Line
-	3000 4500 2650 4500
+	2650 4500 3000 4500
+Wire Wire Line
+	3000 4500 3350 4500
 Wire Wire Line
 	3650 6100 3775 6100
@@
 P 2300 1950
 F 0 "R10" V 2380 1950 50  0000 C CNN
-F 1 "R" V 2300 1950 50  0000 C CNN
+F 1 "200" V 2300 1950 50  0000 C CNN
 F 2 "" H 2300 1950 60  0000 C CNN
 F 3 "" H 2300 1950 60  0000 C CNN
@@
 Wire Wire Line
 	3200 5150 3300 5150
+Text Label 3850 4900 0    60   ~ 0
+SCL
+Wire Wire Line
+	2950 4400 2650 4400
+Connection ~ 3000 4500
+Text Label 3850 5000 0    60   ~ 0
+SDA
+Text Notes 2600 950  0    60   ~ 0
+        R =  340V / 1A\n--------------------\n(1A - opto triac max surge current)
+Text Notes -250 3700 0    60   ~ 0
+TODO: move ON signal to another pin, ICP is cool for capturing timer
 $EndSCHEMATC

Commit message: Change ZC detection subcircuit to a more efficient one, add BOM data to schematics, Also a new kicad
Parts:
- removed U3: LTV-814, ~, symbol OPTO-TRANSISTOR-AC
- added C7: 10u, symbol CP
- added C8: 1n, symbol C
- added D3, D4, D5, D6, D7: 1N4148, Diodes_SMD:SOD-323, symbol D
- added Q2: 2N3904, w_smd_trans:sot23, symbol Q_NPN_BCE
- added R13, R14: 220k, w_smd_resistors:r_1206, symbol R
- added U3: 4N25, optocoupler-2-SO-4, symbol 4N25
- C1: footprint (none) -> rc-master-C100-140X060; symbol C -> C-RESCUE-ssr; Distributor (none) -> Digikey/399-9641-ND; Manufacturer (none) -> Kemet; PartNo (none) -> R46KF210050N0K
- C2: footprint (none) -> rc-master-C150-190X070; symbol C -> C-RESCUE-ssr; Distributor (none) -> Digikey/399-5459-ND; Manufacturer (none) -> Kemet; PartNo (none) -> R46KI24700001K1
- C3: footprint (none) -> rc-master-C150-190X070; symbol C -> C-RESCUE-ssr; Distributor (none) -> Digikey/P11006-ND; Manufacturer (none) -> Panasonic Electronic Components; PartNo (none) -> ECQ-U2A124ML
- C4: footprint (none) -> -C0603; symbol C -> C-RESCUE-ssr
- C5: footprint (none) -> rc-master-CE-035X100
- C6: footprint ~ -> c_0603; symbol C -> C-RESCUE-ssr; Distributor (none) -> ?; Manufacturer (none) -> ?; PartNo (none) -> ?
- CON1: footprint AVR-ISP-6 -> atmel-AVR-ISP-6; symbol AVR-ISP-6 -> AVR-ISP-6-RESCUE-ssr; Distributor (none) -> ?; Manufacturer (none) -> ?; PartNo (none) -> ?
- D1, D2: footprint ~ -> SM0805; symbol LED -> LED-RESCUE-ssr; Distributor (none) -> ?; Manufacturer (none) -> ?; PartNo (none) -> ?
- F1: footprint (none) -> Fuseholder5x20_horiz_open_universal_Type-III; Distributor (none) -> F4830-ND; Manufacturer (none) -> Littelfuse Inc.; PartNo (none) -> 0314030.MXP
- IC1: footprint SO14 -> -SO-14; Distributor (none) -> ?; Manufacturer (none) -> ?; PartNo (none) -> ?
- L1: footprint (none) -> Choke_Toroid_8x16mm_Vertical; Distributor (none) -> ?; Manufacturer (none) -> ?; PartNo (none) -> ?
- P1, P6: footprint (none) -> connect-SC-04; Distributor (none) -> ?; Manufacturer (none) -> ?; PartNo (none) -> ?
- P2, P3, P4: footprint ~ -> HOLE_60; Distributor (none) -> ?; Manufacturer (none) -> ?; PartNo (none) -> ?
- Q1: footprint (none) -> -SOT23; Distributor (none) -> ?; Manufacturer (none) -> ?; PartNo (none) -> ?
- R1: footprint (none) -> Resistor_Horizontal_RM20mm; symbol R -> R-RESCUE-ssr; Distributor (none) -> Digikey/A105915CT-ND; Manufacturer (none) -> TE Connectivity AMP Connectors; PartNo (none) -> 4-1625892-4
- R10, R11, R12, R7, R9: footprint (none) -> w_smd_resistors:r_0603; symbol R -> R-RESCUE-ssr; Distributor (none) -> ?; Manufacturer (none) -> ?; PartNo (none) -> ?
- R2: value 47k -> 4.7k; footprint (none) -> w_smd_resistors:r_0603; Distributor (none) -> ?; Manufacturer (none) -> ?; PartNo (none) -> ?
- R3: footprint (none) -> Resistor_Horizontal_RM15mm; symbol R -> R-RESCUE-ssr; Distributor (none) -> Digikey/39W-1-ND; Manufacturer (none) -> Yageo; PartNo (none) -> RSF100JB-73-39R
- R4: value 16.4k -> 1k; footprint (none) -> w_smd_resistors:r_0603; Distributor (none) -> ?; Manufacturer (none) -> ?; PartNo (none) -> ?
- R5: value 16.4k -> 22k; footprint (none) -> w_smd_resistors:r_0603; Distributor (none) -> ?; Manufacturer (none) -> ?; PartNo (none) -> ?
- R6: footprint (none) -> Resistor_Horizontal_RM15mm; symbol R -> R-RESCUE-ssr; Distributor (none) -> Digikey/A106019CT-ND; Manufacturer (none) -> TE Connectivity AMP Connectors; PartNo (none) -> 1-1625886-8
- R8: footprint (none) -> Resistor_Horizontal_RM15mm; symbol R -> R-RESCUE-ssr; Distributor (none) -> Digikey/S510KHCT-ND; Manufacturer (none) -> Stackpole Electronics Inc.; PartNo (none) -> CFM12JT510K
- U1: footprint (none) -> optocoupler-2-DIL06; symbol OPTO-TRIAC -> OPTO-TRIAC-RESCUE-ssr; Distributor (none) -> Digikey/160-1883-ND; Manufacturer (none) -> Lite-On Inc.; PartNo (none) -> MOC3052
- U2: footprint (none) -> -TOP3; Distributor (none) -> Digikey/497-2431-5-ND; Manufacturer (none) -> STMicroelectronics; PartNo (none) -> BTA41-600BRG
- VR1: footprint (none) -> varistor-S05K40; Distributor (none) -> Dikigey/MOV-07D431K-ND; Manufacturer (none) -> Bourns Inc.; PartNo (none) -> MOV-07D431K
Connections:
- wire segments 97 -> 91
Other:
- note added: "Saugiklio laikiklis:\n\nMFG:Littelfuse Inc. 01220090Z\nFUSE CLIP CARTRIDGE 250V 30A PCB\n\nDigikey/F4190-ND\n\n"
