File: ssr.sch (KiCad schematic (older format))
At the start: 44 parts, among them CON1 AVR-ISP-6, IC1 ATTINY44-SS, P1 CONN_4, P2 CONTACT, P3 CONTACT, P4 CONTACT, P6 CONN_4, Q1 MOSFET_N, Q2 2N3904, U1 MOC-3052, U2 BTA41, U3 4N25

Commit message: Change MCU to attiny441, add rs485, change board dimensions to half-euro-pannel, change leds to THT, change connectors, total reroute
Parts:
- removed IC1: ATTINY44-SS, -SO-14, symbol ATTINY44-SS
- removed P2, P3, P4: CONTACT, HOLE_60, symbol CONTACT
- removed Q1: MOSFET_N, -SOT23, symbol MOSFET_N
- added C9: 1u, Capacitors_SMD:C_0603, symbol C-RESCUE-ssr
- added CONN10: CONN_01X06, Pin_Headers:Pin_Header_Straight_1x06_Pitch2.54mm, symbol CONN_01X06
- added IC2: ATTINY441-SSU, Housings_SOIC:SOIC-14_3.9x8.7mm_Pitch1.27mm, symbol ATTINY441-SSU
- added J1: 240VAC, Connectors_Molex:Molex_MiniFit-JR-5556-02A_2x01x4.20mm_Straight, symbol CONN_01X02
- added J2: LOAD, Connectors_Molex:Molex_MiniFit-JR-5556-02A_2x01x4.20mm_Straight, symbol CONN_01X02
- added Q1: 2N3904, w_smd_trans:sot23, symbol Q_NPN_BCE
- added R15: 1k, w_smd_resistors:r_0603, symbol R
- added R16: 0R, w_smd_resistors:r_0603, symbol R
- added R17: 120, w_smd_resistors:r_0603, symbol R
- added U4: SP3485EN, Housings_SOIC:SOIC-8_3.9x4.9mm_Pitch1.27mm, symbol SP3485EN
- C1: footprint rc-master-C100-140X060 -> Capacitors_ThroughHole:C_Rect_L13_W4_P10; Distributor Digikey/399-9641-ND -> Farnell/1679293
- C2: footprint rc-master-C150-190X070 -> Capacitors_ThroughHole:C_Rect_L13_W6_H12_P10; Distributor Digikey/399-5459-ND -> Farnell/1679306; PartNo R46KI24700001K1 -> R46KI24705001K
- C3: footprint rc-master-C150-190X070 -> Capacitors_ThroughHole:C_Rect_L13_W6_H12_P10; Distributor Digikey/P11006-ND -> Farnell/1413837; Manufacturer Panasonic Electronic Components -> VISHAY BC COMPONENTS; PartNo ECQ-U2A124ML -> BFC233922104
- C4: value 100nF -> 1u; footprint -C0603 -> Capacitors_SMD:C_0603; Distributor (none) -> ?; Manufacturer (none) -> ?; PartNo (none) -> ?
- C5: footprint rc-master-CE-035X100 -> Capacitors_Elko_ThroughHole:Elko_vert_11.2x7.5mm_RM2.5_CopperClear; Distributor (none) -> ?; Manufacturer (none) -> ?; PartNo (none) -> ?
- C6: footprint c_0603 -> Capacitors_SMD:C_0603
- C7: footprint (none) -> Capacitors_Elko_ThroughHole:Elko_vert_11.2x7.5mm_RM2.5_CopperClear; symbol CP -> CP-RESCUE-ssr; Distributor (none) -> ?; Manufacturer (none) -> ?; PartNo (none) -> ?
- C8: footprint (none) -> w_smd_cap:c_0603; Distributor (none) -> ?; Manufacturer (none) -> ?; PartNo (none) -> ?
- CON1: footprint atmel-AVR-ISP-6 -> Pin_Headers:Pin_Header_Straight_2x03_Pitch2.54mm
- F1: Distributor F4830-ND -> Farnell/1596783
- Q2: Distributor ? -> Farnell/1773602; Manufacturer ? -> DIODES INC.; PartNo ? -> MMBT3904-7-F
- R1: footprint Resistor_Horizontal_RM20mm -> w_pth_resistors:R15.5x6; Distributor Digikey/A105915CT-ND -> Farnell/2329590; Manufacturer TE Connectivity AMP Connectors -> TE CONNECTIVITY; PartNo 4-1625892-4 -> CFR200J390R
- R11, R12: value R -> 220
- R13: footprint w_smd_resistors:r_1206 -> w_smd_resistors:r_2010; Distributor Farnell/2447485 -> Farnell/1887681RL; PartNo MCWR12X2203FTL -> MCPWR10FTEQ2203
- R14: footprint w_smd_resistors:r_1206 -> w_smd_resistors:r_2010; Distributor ? -> Farnell/1887681RL; PartNo MCWR12X2203FTL -> MCPWR10FTEQ2203
- R3: footprint Resistor_Horizontal_RM15mm -> w_pth_resistors:RC05; Distributor Digikey/39W-1-ND -> Farnell/1565385; Manufacturer Yageo -> WELWYN; PartNo RSF100JB-73-39R -> MFP1-39R JI
- R6: footprint Resistor_Horizontal_RM15mm -> w_pth_resistors:R12x5.2; Distributor Digikey/A106019CT-ND -> Farnell/2329459; Manufacturer TE Connectivity AMP Connectors -> TE CONNECTIVITY; PartNo 1-1625886-8 -> CFR100J470R
- R7: value R -> 10k
- R8: footprint Resistor_Horizontal_RM15mm -> w_pth_resistors:RC05; Distributor Digikey/S510KHCT-ND -> Farnell/9340700; Manufacturer Stackpole Electronics Inc. -> MULTICOMP; PartNo CFM12JT510K -> MF50 510K
- U1: Distributor Digikey/160-1883-ND -> Farnell/1086680; Manufacturer Lite-On Inc. -> FAIRCHILD SEMICONDUCTOR; PartNo MOC3052 -> MOC3052M
- U2: footprint -TOP3 -> w_to:top3; Distributor Digikey/497-2431-5-ND -> Farnell/1057288
- U3: value 4N25 -> 4N35; footprint optocoupler-2-SO-4 -> w_smd_dil:mdip_6; Distributor ? -> Farnell/1021179; Manufacturer ? -> FAIRCHILD SEMICONDUCTOR; PartNo ? -> 4N35S-M..
- VR1: Distributor Dikigey/MOV-07D431K-ND -> Farnell/1856861; Manufacturer Bourns Inc. -> MULTICOMP; PartNo MOV-07D431K -> MCSR431K07DS
Connections:
- net GND: now also P6.4 (P4), C9.2, CONN10.1 (P1), IC2.14 (GND), Q1.3 (E), U4.5 (GND); no longer P6.1 (P1)
- net LINE: now also VR1.1
- net MISO: now also R12.1, IC2.8 ((PCINT5/MISO/TXD1/T2/TOCC4/ACO0/ADC5)PA5)
- net MOSI: now also R11.1, IC2.7 ((PCINT6/MOSI/SDA/XCK1/TOCC5/ACO1/ADC6)PA6); no longer P6.3 (P3)
- net NEUTRAL: now also J1.2 (P2), J2.2 (P2)
- net ON: now also P1.3 (P3), IC2.2 ((PCINT8/CLKI/XTAL1/ADC11)PB0), R15.1; no longer P1.2 (P2)
- net RESET: now also IC2.4 ((PCINT11/dW/~RESET~/ADC9)PB3)
- net SCK: now also IC2.9 ((PCINT4/SCK/SCL/RXD1/T1/TOCC3/AIN11/ADC4)PA4), U4.2 (~RE~), U4.3 (DE); no longer P6.2 (P2)
- net VCC: now also P1.2 (P2), P6.1 (P1), C9.1, CONN10.6 (P6), IC2.1 (VCC), U4.8 (VCC); no longer P1.3 (P3), P6.4 (P4)
- net ZERO_CROSSING: now also IC2.3 ((PCINT9/INT0/XTAL2/ADC10)PB1)
- net LOAD: now reaches C1.2, C2.2, L1.1, U2.1
- net at C3.1, F1.2, R8.1: now also J1.1 (P1); no longer VR1.1
- net LOAD-FILTERED: now reaches C3.2, L1.2, R8.2
- net LOAD-FILTERED: now also J2.1 (P1)
- net at R10.2: now also Q1.2 (C)
- net at D4.1 (K), D5.1 (K), R4.2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: now also C7.1
- net at C7.2: now also D3.2 (A), Q2.3 (E)
- new net: CONN10.2 (P2), IC2.10 ((PCINT3/SCK/XCK0/T0/TOCC2/AIN10/ADC3)PA3)
- new net: CONN10.3 (P3), IC2.11 ((PCINT2/~SS~/RXD0/TOCC1/AIN01/ADC2)PA2)
- new net: CONN10.4 (P4), IC2.12 ((PCINT1/MOSI/TXD0/TOCC0/AIN00/ADC1)PA1)
- new net: CONN10.5 (P5), IC2.13 ((PCINT0/MISO/AREF/ADC0)PA0)
- new net: Q1.1 (B), R15.2
- new net: R16.2, R17.1
- new net RS485-A: P6.3 (P3), R16.1, U4.6 (A)
- new net RS485-B: P6.2 (P2), R17.2, U4.7 (B)
- new net RX: IC2.5 ((PCINT10/RXD0/ICP2/CLKO/TOCC7/ADC8)PB2), U4.1 (RO)
- new net TX: IC2.6 ((PCINT7/~SS~/TXD0/ICP1/TOCC6/ADC7)PA7), U4.4 (DI)
Other:
- note added: "Saugiklio laikiklis:\n\nMFG:Littelfuse Inc. 01220090Z\nFUSE CLIP CARTRIDGE 250V 30A PCB\n\nDigikey/F4190-ND\nFarnell/1608255\n0.87€\n"
- note removed: "240VAC"
- note removed: "LOAD"
- note removed: "Saugiklio laikiklis:\n\nMFG:Littelfuse Inc. 01220090Z\nFUSE CLIP CARTRIDGE 250V 30A PCB\n\nDigikey/F4190-ND\n\n"
- moved on the sheet: C4, C5, C7, C8, CON1, D1, D2, D3, D4, D5, D6, D7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

Commit message: KiCad library change, export PDF schematics
Parts:
- C1, C2, C3, C4, C6, C9: symbol C-RESCUE-ssr -> ssr-rescue:C-RESCUE-ssr
- C7: symbol CP-RESCUE-ssr -> ssr-rescue:CP-RESCUE-ssr
- C8: symbol C -> ssr-rescue:C
- CON1: symbol AVR-ISP-6-RESCUE-ssr -> ssr-rescue:AVR-ISP-6-RESCUE-ssr
- CONN10: symbol CONN_01X06 -> ssr-rescue:CONN_01X06
- D1, D2: symbol LED-RESCUE-ssr -> ssr-rescue:LED-RESCUE-ssr
- D3, D4, D5, D6, D7: symbol D -> ssr-rescue:D
- F1: symbol FUSE -> ssr-rescue:FUSE
- IC2: symbol ATTINY441-SSU -> ssr-rescue:ATTINY441-SSU
- J1, J2: symbol CONN_01X02 -> ssr-rescue:CONN_01X02
- L1: symbol INDUCTOR -> ssr-rescue:INDUCTOR
- P1, P6: symbol CONN_4 -> ssr-rescue:CONN_4
- Q1, Q2: symbol Q_NPN_BCE -> ssr-rescue:Q_NPN_BCE
- R1, R10, R11, R12, R3, R6, R7, R8, R9: symbol R-RESCUE-ssr -> ssr-rescue:R-RESCUE-ssr
- R13, R14, R15, R16, R17, R2, R4, R5: symbol R -> ssr-rescue:R
- U1: symbol OPTO-TRIAC-RESCUE-ssr -> ssr-rescue:OPTO-TRIAC-RESCUE-ssr
- U2: symbol TRIAC -> ssr-rescue:TRIAC
- U3: symbol 4N25 -> ssr-rescue:4N25
- VR1: symbol VR -> ssr-rescue:VR
Other:
- note added: "Zerro Cossing circuit by Dego\nhttp://www.dextrel.net/diyzerocrosser.htm"
